Commit message: fix robot dimensions + add color to robot in simulation + readjust the laser height

File: urdf/barista_robot_model.urdf (robot description, URDF)
Before this commit: robot barista_bot, 8 links, 7 joints
Links:
- link chassis: geometry collision cylinder length=0.090 radius=0.160; collision cylinder length=0.155 radius=0.178
- link left_wheel: geometry collision cylinder length=0.0106 radius=0.0352; visual cylinder length=0.0106 radius=0.0352
- link right_wheel: geometry collision cylinder length=0.0106 radius=0.0352; visual cylinder length=0.0106 radius=0.0352
Joints:
- joint back_cater_wheel_joint: origin xyz=-0.25 0 -0.0775 rpy=0 0 0 -> xyz=-0.125 0 -0.0775 rpy=0 0 0
- joint front_caster_wheel_joint: origin xyz=0.25 0 -0.0775 rpy=0 0 0 -> xyz=0.125 0 -0.0775 rpy=0 0 0
- joint hokuyo_laser_joint: origin xyz=0.3 0 0.0775 rpy=0 0 0 -> xyz=0.15 0 0.0775 rpy=0 0 0
- joint left_wheel_joint: origin xyz=0 0.25 -0.0775 rpy=0 0 0 -> xyz=0 0.125 -0.0775 rpy=0 0 0
- joint right_wheel_joint: origin xyz=0 -0.25 -0.0775 rpy=0 0 0 -> xyz=0 -0.125 -0.0775 rpy=0 0 0
