Commit message: fixing robot dimension error from the xacro file

File: xacro/barista_robot_model.urdf.xacro (robot description, xacro)
@@ -8,5 +8,5 @@
   <xacro:include filename="$(find barista_robot_description)/xacro/gazebo.xacro"/>
   <xacro:property name="chassis_length" value="0.155"/>
-  <xacro:property name="chassis_radius" value="0.356"/>
+  <xacro:property name="chassis_radius" value="0.178"/>
   <xacro:property name="chassis_mass" value="5"/>
   <material name="grey">
@@ -18,4 +18,7 @@
   <material name="blue">
     <color rgba="0.2 0.1 0.8 1"/>
+  </material>
+  <material name="red">
+    <color rgba="0.8 0.1 0.2 1"/>
   </material>
   <link name="base_link">
@@ -33,5 +36,5 @@
         <cylinder length="${chassis_length}" radius="${chassis_radius}"/>
       </geometry>
-      <material name="grey"/>
+      <material name="blue"/>
     </visual>
     <collision>
@@ -46,10 +49,13 @@
       <inertia ixx="0.16843041666666667" ixy="0" ixz="0" iyy="0.16843041666666667" iyz="0" izz="0.31683999999999996"/>
     </inertial>
-    <xacro:standoff pos_x="0.050" pos_y="0.250" pos_z="0.1875"/>
-    <xacro:standoff pos_x="-0.050" pos_y="0.250" pos_z="0.1875"/>
-    <xacro:standoff pos_x="0.050" pos_y="-0.250" pos_z="0.1875"/>
-    <xacro:standoff pos_x="-0.050" pos_y="-0.250" pos_z="0.1875"/>
+    <xacro:standoff pos_x="0.025" pos_y="0.100" pos_z="0.1875"/>
+    <xacro:standoff pos_x="-0.025" pos_y="0.100" pos_z="0.1875"/>
+    <xacro:standoff pos_x="0.025" pos_y="-0.100" pos_z="0.1875"/>
+    <xacro:standoff pos_x="-0.025" pos_y="-0.100" pos_z="0.1875"/>
     <xacro:cup_holder_tray />
   </link>
+  <gazebo reference="chassis">
+    <material>Gazebo/Blue</material>
+  </gazebo>
   <xacro:caster_wheel caster_wheel_name="front_caster_wheel" side="1"/>
   <xacro:caster_wheel caster_wheel_name="back_caster_wheel" side="-1"/>
@@ -58,5 +64,5 @@
   <xacro:if value="${include_laser}">
     <joint name="hokuyo_laser_joint" type="fixed">
-      <origin xyz="0.3 0 0.0775" rpy="0 0 0"/>
+      <origin xyz="0.15 0 0.0775" rpy="0 0 0"/>
       <parent link="chassis"/>
       <child link="hokuyo_laser"/>
@@ -68,4 +74,5 @@
           <mesh filename="package://barista_robot_description/meshes/hokuyo_urg_04lx.dae" scale="1.0 1.0 1.0"/>
         </geometry>
+        <material name="black"/>
       </visual>
       <collision>

File: xacro/caster_wheel.xacro (robot description, xacro)
@@ -7,5 +7,5 @@
     "side" 1 for front caster wheel, -1 for back caster wheel -->
     <joint name="${caster_wheel_name}_joint" type="fixed">
-      <origin xyz="${side * 0.25} 0 -0.0775" rpy="0 0 0"/>
+      <origin xyz="${side * 0.125} 0 -0.0775" rpy="0 0 0"/>
       <parent link="chassis"/>
       <child link="${caster_wheel_name}"/>
@@ -17,5 +17,5 @@
         <sphere radius="0.0352"/>
       </geometry>
-      <material name="blue"/>
+      <material name="red"/>
     </visual>
     <collision>
@@ -36,5 +36,5 @@
     <mu1>0.1</mu1>
     <mu2>0.1</mu2>
-    <material>Gazebo/Blue</material>
+    <material>Gazebo/Red</material>
   </gazebo>
   </xacro:macro>

File: xacro/cup_holder_tray.xacro (robot description, xacro)
@@ -6,5 +6,5 @@
       <origin xyz="0 0 0.3425" rpy="0 0 0"/>
       <geometry>
-        <cylinder length="0.090" radius="0.320"/>
+        <cylinder length="0.090" radius="0.160"/>
       </geometry>
     </visual>
@@ -12,5 +12,5 @@
       <origin xyz="0 0 0.3425" rpy="0 0 0"/>
       <geometry>
-        <cylinder length="0.090" radius="0.320"/>
+        <cylinder length="0.090" radius="0.160"/>
       </geometry>
     </collision>

File: xacro/gazebo.xacro (robot description, xacro)
@@ -32,4 +32,7 @@
   <xacro:if value="${include_laser}">
     <gazebo reference="laser_scan_frame">
+      <material>Gazebo/Black</material>
+    </gazebo>
+    <gazebo reference="laser_scan_frame">
       <sensor name="sensor_ray" type="ray">
           <pose>0 0 0 0 0 0</pose>
@@ -45,5 +48,5 @@
             <range>
               <min>0.1</min>
-              <max>15.0</max>
+              <max>5.0</max>
             </range>
           </ray>
@@ -53,8 +56,8 @@
           <plugin name="laser" filename="libgazebo_ros_ray_sensor.so">
             <ros>
-              <namespace>/barista_bot</namespace>
               <remapping>~/out:=scan</remapping>
             </ros>
             <output_type>sensor_msgs/LaserScan</output_type>
+            <frame_name>laser_scan_frame</frame_name>
           </plugin>
       </sensor>

File: xacro/standoff.xacro (robot description, xacro)
@@ -5,5 +5,5 @@
       <origin xyz="${pos_x} ${pos_y} ${pos_z}" rpy="0 0 0"/>
       <geometry>
-        <cylinder length="0.220" radius="0.020"/>
+        <cylinder length="0.220" radius="0.010"/>
       </geometry>
     </visual>
@@ -11,5 +11,5 @@
       <origin xyz="${pos_x} ${pos_y} ${pos_z}" rpy="0 0 0"/>
       <geometry>
-        <cylinder length="0.220" radius="0.020"/>
+        <cylinder length="0.220" radius="0.010"/>
       </geometry>
     </collision>

File: xacro/wheel.xacro (robot description, xacro)
@@ -8,5 +8,5 @@
     "side" 1 for left wheel, -1 for right wheel -->
     <joint name="${wheel_name}_joint" type="continuous">
-      <origin xyz="0 ${side * 0.25} -0.0775" rpy="0 0 0"/>
+      <origin xyz="0 ${side * 0.125} -0.0775" rpy="0 0 0"/>
       <parent link="${ref_frame}"/>
       <child link="${wheel_name}"/>

Commit message: creation of a launch file to spawn two barista_bot

File: xacro/barista_robot_model.urdf.xacro (robot description, xacro)
@@ -1,4 +1,6 @@
 <?xml version="1.0"?>
 <robot xmlns:xacro="http://www.ros.org/wiki/xacro" name="barista_bot">
+  <xacro:arg name="robot_name" default="barista_bot"/>
+  <xacro:property name="robot_name" value="$(arg robot_name)"/>
   <xacro:include filename="$(find barista_robot_description)/xacro/standoff.xacro"/>
   <xacro:include filename="$(find barista_robot_description)/xacro/cup_holder_tray.xacro"/>

File: xacro/gazebo.xacro (robot description, xacro)
@@ -4,4 +4,5 @@
     <plugin name="barista_bot_joint_state" filename="libgazebo_ros_joint_state_publisher.so">
     <ros>
+        <namespace>/${robot_name}</namespace>
         <remapping>~/out:=joint_states</remapping>
     </ros>
@@ -14,4 +15,7 @@
   <gazebo>
     <plugin filename="libgazebo_ros_diff_drive.so" name="differential_drive_controller">
+      <ros>
+        <namespace>/${robot_name}</namespace>
+      </ros>
       <!-- wheels -->
       <left_joint>left_wheel_joint</left_joint>
@@ -26,6 +30,6 @@
       <publish_odom>true</publish_odom>
       <publish_odom_tf>true</publish_odom_tf>
-      <odometry_frame>odom</odometry_frame>
-      <robot_base_frame>base_link</robot_base_frame>
+      <odometry_frame>${robot_name}/odom</odometry_frame>
+      <robot_base_frame>${robot_name}/base_link</robot_base_frame>
     </plugin>
   </gazebo>
@@ -56,8 +60,9 @@
           <plugin name="laser" filename="libgazebo_ros_ray_sensor.so">
             <ros>
+              <namespace>/${robot_name}</namespace>
               <remapping>~/out:=scan</remapping>
             </ros>
             <output_type>sensor_msgs/LaserScan</output_type>
-            <frame_name>laser_scan_frame</frame_name>
+            <frame_name>${robot_name}/laser_scan_frame</frame_name>
           </plugin>
       </sensor>

Commit message: add different color for the robots

File: xacro/barista_robot_model.urdf.xacro (robot description, xacro)
@@ -1,6 +1,7 @@
 <?xml version="1.0"?>
 <robot xmlns:xacro="http://www.ros.org/wiki/xacro" name="barista_bot">
-  <xacro:arg name="robot_name" default="barista_bot"/>
-  <xacro:property name="robot_name" value="$(arg robot_name)"/>
+  <xacro:arg name="r_n" default="barista_bot"/>
+  <xacro:property name="robot_name" value="$(arg r_n)"/>
+  <xacro:property name="morty" value="morty"/>
   <xacro:include filename="$(find barista_robot_description)/xacro/standoff.xacro"/>
   <xacro:include filename="$(find barista_robot_description)/xacro/cup_holder_tray.xacro"/>
@@ -38,5 +39,10 @@
         <cylinder length="${chassis_length}" radius="${chassis_radius}"/>
       </geometry>
+      <xacro:if value="${robot_name == morty}">
       <material name="blue"/>
+      </xacro:if>
+      <xacro:unless value="${robot_name == morty}">
+      <material name="red"/>
+      </xacro:unless>
     </visual>
     <collision>
@@ -57,7 +63,14 @@
     <xacro:cup_holder_tray />
   </link>
+  <xacro:if value="${robot_name == morty}">
   <gazebo reference="chassis">
     <material>Gazebo/Blue</material>
   </gazebo>
+  </xacro:if>
+  <xacro:unless value="${robot_name == morty}">
+  <gazebo reference="chassis">
+    <material>Gazebo/Red</material>
+  </gazebo>
+  </xacro:unless>
   <xacro:caster_wheel caster_wheel_name="front_caster_wheel" side="1"/>
   <xacro:caster_wheel caster_wheel_name="back_caster_wheel" side="-1"/>

File: xacro/caster_wheel.xacro (robot description, xacro)
@@ -17,5 +17,5 @@
         <sphere radius="0.0352"/>
       </geometry>
-      <material name="red"/>
+      <material name="grey"/>
     </visual>
     <collision>
@@ -36,5 +36,5 @@
     <mu1>0.1</mu1>
     <mu2>0.1</mu2>
-    <material>Gazebo/Red</material>
+    <material>Gazebo/Grey</material>
   </gazebo>
   </xacro:macro>
